File: merope-pcb/merope-central/merope-central.brd (EAGLE design)
At the start: 100 x 80 mm, 26 parts, among them IC1 PCF8563, IC2 MICROSD-UP, IC3 MEGA48/88/168-AU, IC4 HC-05_VER2, X1 TERMINAL_BLOCK_35_2, X2 TERMINAL_BLOCK_35_2, X3 TERMINAL_BLOCK_35_2, X4 TERMINAL_BLOCK_35_2, X5 TERMINAL_BLOCK_35_2, X6 TERMINAL_BLOCK_35_2, X7 TERMINAL_BLOCK_35_2, X8 TERMINAL_BLOCK_35_2

Commit message: Added some files and changed some information.
Other:
- board text added: "Merope-Power (C) 2014-2016 Erik Kos"
- board text removed: "Merope-Power (C) 2014-2016 Jacek Szymoniak"
Changed lines of the file:
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@@
 <text x="68.8975" y="19.3675" size="0.8128" layer="25">Merope-Power
 (C) 2014-2016
-Jacek Szymoniak</text>
+Erik Kos</text>
 </plain>
 <attributes>
