File: merope-pcb/merope-central/merope-central.sch (EAGLE design)
At the start: 25 parts, among them IC1 PCF8563, IC2 MICROSD-UP, IC3 MEGA48/88/168-AU, IC4 HC-05_VER2, X1 TERMINAL_BLOCK_35_2, X2 TERMINAL_BLOCK_35_2, X3 TERMINAL_BLOCK_35_2, X4 TERMINAL_BLOCK_35_2, X5 TERMINAL_BLOCK_35_2, X6 TERMINAL_BLOCK_35_2, X7 TERMINAL_BLOCK_35_2, X8 TERMINAL_BLOCK_35_2

Commit message: Added some files and changed some information.
Other:
- note added: "Copyright (C) 2014-2016 Erik Kos License: Creative Commons Attribution-ShareAlike 4.0"
- note removed: "Copyright (C) 2014-2016 Jacek Szymoniak License: Creative Commons Attribution-ShareAlike 4.0"
Changed lines of the file:
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@@
 <sheet>
 <plain>
-<text x="167.64" y="25.4" size="2.794" layer="94">Copyright (C) 2014-2016 Jacek Szymoniak
+<text x="167.64" y="25.4" size="2.794" layer="94">Copyright (C) 2014-2016 Erik Kos
 License: Creative Commons Attribution-ShareAlike 4.0</text>
 </plain>
