File: merope-pcb/merope-power/merope-power.brd (EAGLE design)
At the start: 100 x 80 mm, 20 parts, among them IC1 78L05F, IC2 78L05F, IC3 TS520533, X1 TERMINAL_BLOCK_5_2, X2 TERMINAL_BLOCK_35_2, X3 TERMINAL_BLOCK_35_2, X4 TERMINAL_BLOCK_35_2, X5 TERMINAL_BLOCK_35_2, X6 TERMINAL_BLOCK_35_2, X7 TERMINAL_BLOCK_35_2

Commit message: Added some files and changed some information.
Other:
- board text added: "Merope-Power (C) 2014-2016 Erik Kos"
- board text removed: "Merope-Power (C) 2014-2016 Jacek Szymoniak"
Changed lines of the file:
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@@
 <text x="16.66875" y="15.875" size="1.016" layer="25">Merope-Power
 (C) 2014-2016
-Jacek Szymoniak</text>
+Erik Kos</text>
 </plain>
 <attributes>
