File: merope-pcb/merope-power/merope-power.sch (EAGLE design)
At the start: 19 parts, among them IC1 78L05F, IC2 78L05F, IC3 TS520533, X1 TERMINAL_BLOCK_5_2, X2 TERMINAL_BLOCK_35_2, X3 TERMINAL_BLOCK_35_2, X4 TERMINAL_BLOCK_35_2, X5 TERMINAL_BLOCK_35_2, X6 TERMINAL_BLOCK_35_2, X7 TERMINAL_BLOCK_35_2

Commit message: Added some files and changed some information.
Other:
- note added: "Copyright (C) 2014-2016 Erik Kos License: Creative Commons Attribution-ShareAlike 4.0"
- note removed: "Copyright (C) 2014-2016 Jacek Szymoniak License: Creative Commons Attribution-ShareAlike 4.0"
Changed lines of the file:
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@@
 <plain>
 <text x="63.5" y="-40.64" size="2.794" layer="94">Copyright (C) 2014-2016
-Jacek Szymoniak
+Erik Kos
 License: Creative Commons
 Attribution-ShareAlike 4.0</text>
