File: merope-pcb/merope-relays/merope-relays.sch (EAGLE design)
At the start: 20 parts, among them T1 BC847, T2 BC847, T3 BC847, T4 BC847, X1 TERMINAL_BLOCK_35_2, X10 TERMINAL_BLOCK_35_2, X3 TERMINAL_BLOCK_5_3, X4 TERMINAL_BLOCK_5_2, X5 TERMINAL_BLOCK_35_2, X6 TERMINAL_BLOCK_35_2

Commit message: Added some files and changed some information.
Other:
- note added: "Copyright (C) 2014-2016 Erik Kos License: Creative Commons Attribution-ShareAlike 4.0"
- note removed: "Copyright (C) 2014-2016 Jacek Szymoniak License: Creative Commons Attribution-ShareAlike 4.0"
Changed lines of the file:
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@@
 <plain>
 <text x="35.052" y="-79.756" size="2.794" layer="94">Copyright (C) 2014-2016
-Jacek Szymoniak
+Erik Kos
 License: Creative Commons
 Attribution-ShareAlike 4.0</text>
